Commit message: Update robot.urdf

File: urdf/robot.urdf (robot description, URDF)
Before this commit: robot my_robot, 6 links, 5 joints
Joints:
- removed joint left_back_wheel_joint
- removed joint left_front_wheel_joint
- removed joint right_back_wheel_joint
- removed joint right_front_wheel_joint
- added joint left_back_wheel_joint_differential: type continuous, parent link_chassis, child left_back_wheel, origin xyz=-0.9 0.95 -0.25 rpy=0 0 1.5707, axis 1 0 0, limit effort=100 velocity=100
- added joint left_front_wheel_joint_differential: type continuous, parent link_chassis, child left_front_wheel, origin xyz=0.9 0.95 -0.25 rpy=0 0 1.5707, axis 1 0 0, limit effort=100 velocity=100
- added joint right_back_wheel_joint_differential: type continuous, parent link_chassis, child right_back_wheel, origin xyz=-0.9 -0.95 -0.25 rpy=0 0 1.5707, axis 1 0 0, limit effort=100 velocity=100
- added joint right_front_wheel_joint_differential: type continuous, parent link_chassis, child right_front_wheel, origin xyz=0.9 -0.95 -0.25 rpy=0 0 1.5707, axis 1 0 0, limit effort=100 velocity=100
